File: ladcp_interface_box/ladcp_interface_box/ladcp_interface_box.kicad_sch (KiCad schematic)
At the start: 2 parts, among them J1 TERM BLK 8POS SIDE ENTRY 5MM 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, U1 FT4232H

Commit message: updated files
Parts:
- added C1, C10, C2, C4, C5, C6, C7, C8, C9: .1uF, Capacitor_SMD:C_0805_2012Metric_Pad1.18x1.45mm_HandSolder, symbol Device:C_Small
- added C3: 3.3uF, Capacitor_SMD:C_0805_2012Metric_Pad1.18x1.45mm_HandSolder, symbol Device:C_Small
- added FB1, FB2: FerriteBead_Small, Inductor_SMD:L_0805_2012Metric_Pad1.15x1.40mm_HandSolder, symbol Device:FerriteBead_Small
- added J2: USB_B_Mini, Connector_USB:USB_Mini-B_Wuerth_65100516121_Horizontal, symbol Connector:USB_B_Mini
- added U2: LF33_TO252, Package_TO_SOT_SMD:TO-252-3_TabPin2, symbol Regulator_Linear:LF33_TO252
- added X1: ECS-2033-120-BN, Oscillator:Oscillator_SMD_ECS_2520MV-xxx-xx-4Pin_2.5x2.0mm, symbol Oscillator:ECS-2520MV-xxx-xx
Connections:
- net +1.8V: now reaches U1.12 (VCORE)
- net +1.8V: now also U1.37 (VCORE), U1.49 (VREGOUT), U1.64 (VCORE), C3.1, C4.1, C5.1, C6.1
- net +3.3V: now reaches U1.20 (VCCIO)
- net +3.3V: now also U1.31 (VCCIO), U1.42 (VCCIO), U1.50 (VREGIN), U1.56 (VCCIO), C10.1, C2.1, C7.1, C8.1, C9.1, U2.3 (VO)
- net at U1.7 (DM): now also J2.2 (D-)
- net at U1.8 (DP): now also J2.3 (D+)
- new net: C1.1, J2.1 (VBUS), U2.1 (VI)
- new net GNDD: C1.2, C10.2, C2.2, C3.2, C4.2, C5.2, C6.2, C7.2, C8.2, C9.2, J2.4 (ID), J2.5 (GND), J2.6 (Shield), U2.2 (GND)
Other:
- moved on the sheet: J1, U1

Commit message: added PCB design
Parts:
- added C11, C12, C15, C16, C17, C18, C19: .1uF, Capacitor_SMD:C_0805_2012Metric_Pad1.18x1.45mm_HandSolder, symbol Device:C_Small
- added C13, C14, C20: 4.7uF, Capacitor_Tantalum_SMD:CP_EIA-2012-12_Kemet-R_Pad1.30x1.05mm_HandSolder, symbol Device:C_Polarized_Small
- added H1, H2: MountingHole, MountingHole:MountingHole_2.1mm, symbol Mechanical:MountingHole
- added J3: BATTERY CHARGER GOES HERE., TerminalBlock_Phoenix:TerminalBlock_Phoenix_PT-1,5-2-5.0-H_1x02_P5.00mm_Horizontal, symbol Connector:Screw_Terminal_01x02
- added J4: EXTERNAL SWITCH GOES HERE., TerminalBlock_Phoenix:TerminalBlock_Phoenix_PT-1,5-2-5.0-H_1x02_P5.00mm_Horizontal, symbol Connector:Screw_Terminal_01x02
- added J5: AMMETER GOES HERE, TerminalBlock_Phoenix:TerminalBlock_Phoenix_PT-1,5-2-5.0-H_1x02_P5.00mm_Horizontal, symbol Connector:Screw_Terminal_01x02
- added J6: CONNECT VOLT METER HERE, TerminalBlock_Phoenix:TerminalBlock_Phoenix_PT-1,5-2-5.0-H_1x02_P5.00mm_Horizontal, symbol Connector:Screw_Terminal_01x02
- added R1: 1K, Resistor_SMD:R_0805_2012Metric_Pad1.20x1.40mm_HandSolder, symbol Device:R_Small_US
- added R2: 12K, Resistor_SMD:R_0805_2012Metric_Pad1.20x1.40mm_HandSolder, symbol Device:R_Small_US
- added U3: MAX3232, Package_SO:TSSOP-16_4.4x5mm_P0.65mm, symbol Interface_UART:MAX3232
Connections:
- net DATA_RTN is gone; now on net GNDD: J1.4 (Pin_4)
- net POWER- is gone; now on net GNDD: J1.7 (Pin_7)
- net +3.3V: now also FB1.1, FB2.1, X1.1 (Tri-State), X1.4 (VDD), C11.1, C12.1, C13.1, C14.1, R1.2
- net GNDD: now also U1.1 (GND), U1.10 (AGND), U1.11 (GND), U1.13 (TEST), U1.15 (GND), U1.25 (GND), U1.35 (GND), U1.47 (GND), U1.5 (GND), U1.51 (GND), X1.2 (GND), C11.2, C12.2, C13.2, C14.2, C17.2, C18.2, C20.2, J3.2 (Pin_2), J6.2 (Pin_2), R2.2, U3.15 (GND)
- net RS232_ADCP_IN_MASTER: now also U3.14 (T1OUT)
- net RS232_ADCP_IN_SLAVE: now also U3.7 (T2OUT)
- net RS232_ADCP_OUT_MASTER: now also U3.13 (R1IN)
- net RS232_ADCP_OUT_SLAVE: now also U3.8 (R2IN)
- net at X1.3 (OUT): now also U1.2 (OSCI)
- net at FB1.2: now also U1.4 (VPHY)
- net at FB2.2: now also U1.9 (VPLL)
- net +5V: now reaches C1.1, J2.1 (VBUS), U2.1 (VI)
- net +5V: now also C16.1, C17.1, C20.1, U3.16 (VCC)
- net at U1.14 (~{RESET}): now also R1.1
- net TTL_TX_A: now reaches U1.16 (ADBUS0)
- net TTL_TX_A: now also U3.11 (T1IN)
- net TTL_RX_A: now reaches U1.17 (ADBUS1)
- net TTL_RX_A: now also U3.12 (R1OUT)
- net TTL_TX_B: now reaches U1.26 (BDBUS0)
- net TTL_TX_B: now also U3.10 (T2IN)
- net TTL_RX_B: now reaches U1.27 (BDBUS1)
- net TTL_RX_B: now also U3.9 (R2OUT)
- net at U1.6 (REF): now also R2.1
- net POWER+ renamed +48V
- net +48V: now also J5.1 (Pin_1)
- new net: C19.1, U3.4 (C2+)
- new net: C19.2, U3.5 (C2-)
- new net: C16.2, U3.2 (VS+)
- new net: J3.1 (Pin_1), J4.2 (Pin_2), J6.1 (Pin_1)
- new net: C18.1, U3.6 (VS-)
- new net: C15.1, U3.1 (C1+)
- new net: C15.2, U3.3 (C1-)
- new net: J4.1 (Pin_1), J5.2 (Pin_2)
- no-connect marks 1 -> 35
Other:
- moved on the sheet: FB1, FB2, J1, X1

Commit message: finished circuit
Parts:
- added C21: 50V 1uF, Capacitor_THT:CP_Radial_D4.0mm_P1.50mm, symbol Device:C_Polarized_Small
- added C22: 50V 10uF, Capacitor_THT:CP_Radial_D6.3mm_P2.50mm, symbol Device:C_Polarized_Small
- added J7: +12V, TerminalBlock_Phoenix:TerminalBlock_Phoenix_PT-1,5-2-5.0-H_1x02_P5.00mm_Horizontal, symbol Connector:Screw_Terminal_01x02
- added U5: 12V LDO, Package_TO_SOT_SMD:SOT-23, symbol Regulator_Linear:APE8865N-16-HF-3
- J3: value BATTERY CHARGER GOES HERE. -> CHARGER
- J4: value EXTERNAL SWITCH GOES HERE. -> SWITCH
- J5: value AMMETER GOES HERE -> AMMETER
- J6: value CONNECT VOLT METER HERE -> VOLT METER
- U2: value LF33_TO252 -> 3.3V regulator
- U3: Manufacturer part# MAX3232EUE+T -> (none); Vendor digikey -> (none); Vendor part# MAX3232EUE+TCT-ND -> (none); manufacturer part# (none) -> MAX3232EUE+T; vendor (none) -> digikey; vendor part# (none) -> MAX3232EUE+TCT-ND
Connections:
- net +48V: now also C21.1, U5.3 (VI)
- net GNDD: now also C21.2, C22.2, J7.2 (Pin_2), U5.1 (GND)
- new net +12V: C22.1, J7.1 (Pin_1), U5.2 (VO)
