File: ladcp_interface_box/ladcp_interface_box/ladcp_interface_box.kicad_pcb (KiCad board)
At the start: 2 copper layers, 92 x 41 mm, 36 parts, among them J1 TERM BLK 8POS SIDE ENTRY 5MM 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, J2 USB_B_Mini, J3 BATTERY CHARGER GOES HERE., J4 EXTERNAL SWITCH GOES HERE., J5 AMMETER GOES HERE, J6 CONNECT VOLT METER HERE, U1 FT4232H, U2 LF33_TO252, U3 MAX3232, X1 ECS-2033-120-BN

Commit message: fixed errors
Parts:
- J3: value BATTERY CHARGER GOES HERE. -> CHARGER
- J4: value EXTERNAL SWITCH GOES HERE. -> SWITCH
- J5: value AMMETER GOES HERE -> AMMETER
- J6: value CONNECT VOLT METER HERE -> VOLT METER
- moved C3 3.65 mm to (145.3, 75.9)
- moved C4 3.65 mm to (138.5, 75.9)
- moved C9 3.65 mm to (141.9, 75.9)
Routing:
- net GNDD: track 311.5 -> 73.2 mm, vias 2 -> 16
- net /+48V: track 55.5 -> 123.3 mm
- net /RS232_ADCP_IN_SLAVE: track 50.3 -> 80.3 mm
- net /+1.8V: track 59.5 -> 50.3 mm, vias 5 -> 2
- net /+3.3V: track 154.3 -> 145.9 mm
- net Net-(J4-Pin_1): track 6.55 -> 13.1 mm
- net Net-(J3-Pin_1): track 53.7 -> 60.3 mm

Commit message: finished circuit
Parts:
- added C21: 50V 1uF, Capacitor_THT:CP_Radial_D4.0mm_P1.50mm, F.Cu at (129.8, 99.8)
- added C22: 50V 10uF, Capacitor_THT:CP_Radial_D6.3mm_P2.50mm, F.Cu at (131.8, 105.8)
- added J7: +12V, TerminalBlock_Phoenix:TerminalBlock_Phoenix_PT-1,5-2-5.0-H_1x02_P5.00mm_Horizontal, F.Cu at (165.6, 105.6)
- added U5: 12V LDO, Package_TO_SOT_SMD:SOT-23, F.Cu at (128.6, 96.1)
- U2: value LF33_TO252 -> 3.3V regulator
- X1: value ECS-2033-120-BN -> CRYSTAL
- moved C18 12.2 mm to (160.2, 96.4), turned to 90 degrees
- moved C19 2.13 mm to (154.9, 106.6)
- moved C15 2.11 mm to (149.7, 106.5)
Routing:
- net /+12V: track 0.00 -> 53.5 mm, vias 0 -> 2
- net /+48V: track 123.3 -> 141.7 mm
- net /RS232_ADCP_IN_SLAVE: track 80.3 -> 87.0 mm
- net /+5V: track 89.6 -> 86.0 mm
- net Net-(U3-C1+): track 9.09 -> 6.91 mm
- net Net-(U3-VS-): track 7.28 -> 9.33 mm
- net Net-(U3-C2+): track 5.81 -> 4.06 mm
- net Net-(U3-C2-): track 6.41 -> 5.04 mm
- net /RS232_ADCP_IN_MASTER: track 43.8 -> 44.9 mm
- net Net-(U3-C1-): track 6.72 -> 5.66 mm
- net GNDD: vias 16 -> 18

Commit message: added final changes
Parts:
- added G***: LOGO, ladcp_interface_box:noaa_logo_8x8, F.Cu at (152.6, 75.1)
- added G***: LOGO, ladcp_interface_box:noaa_logo, B.Cu at (151.1, 85.3)
Other:
- board text added: "Pedro Pena"
- board text added: "Rev 1.0.0"
