File: ladcp_star_circuit/ladcp_star_circuit.kicad_pcb (KiCad board)
At the start: 2 copper layers, 48.3 x 88.9 mm, 9 parts, among them P1 TERM BLK 8POS SIDE ENTRY 5MM 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, P2 TERM BLK 8POS SIDE ENTRY 5MM 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, P3 TERM BLK 2POS SIDE ENTRY 5MM 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, P6 TERM BLK 8POS SIDE ENTRY 5MM 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

Commit message: added final changes
Parts:
- added G***: LOGO, ladcp_star_circuit:noaa_logo, F.Cu at (136.4, 124.0)
Other:
- board text added: "LADCP Star-board"
- board text added: "Star Board. LADCP Star Cable Replacement Rev 1.0.0 Pedro Pena"
- board text removed: "Star Board. LADCP Star Cable Replacement Rev 1.0.0"
